Commit message: add wheel-biped robot

File: legged_gym/resources/robots/bigreddog/urdf/big_reddog.urdf (robot description, URDF)
Before this commit: robot big_reddog, 35 links, 34 joints
Joints:
- joint FL_hip_joint: limit lower=-0.61 upper=0.61 effort=80.0 velocity=20. -> lower=-1.0472 upper=1.0472 effort=80.0 velocity=20.
- joint FR_hip_joint: limit lower=-0.61 upper=0.61 effort=80.0 velocity=20. -> lower=-1.0472 upper=1.0472 effort=80.0 velocity=20.
- joint RL_hip_joint: limit lower=-0.61 upper=0.61 effort=80.0 velocity=20. -> lower=-1.0472 upper=1.0472 effort=80.0 velocity=20.
- joint RR_hip_joint: limit lower=-0.61 upper=0.61 effort=80.0 velocity=20. -> lower=-1.0472 upper=1.0472 effort=80.0 velocity=20.
